File: mario2.kicad_pcb (KiCad board)
At the start: 2 copper layers, 38.1 x 40.6 mm, 7 parts, among them J1 Resistors, J2 FSRs, U1 Teensy-LC

Commit message: Clean up schematic wiring
Connections:
- net Net-(J1-Pad1) renamed GND
- net Net-(J1-Pad2) renamed /FSR_1
- net Net-(J1-Pad4) renamed /FSR_2
- net Net-(J1-Pad6) renamed /FSR_3
- net Net-(J1-Pad8) renamed /FSR_4
- net Net-(J2-Pad1) renamed +3V3
